File: PCB/Sensor_Board/Sensor_Board.kicad_pcb (KiCad board)
At the start: 2 copper layers, 90 x 90 mm, 7 parts, among them J1 Conn_01x08_Socket, J2 Conn_01x06_Socket, J3 Conn_01x04_Socket, J4 Conn_01x07_Socket, J5 Conn_01x09_Socket, J6 SE2-30

Commit message: updated footprint from lib
Parts:
- removed G***: LOGO, SE2-30:Rocketry_Logo_Symbol
Other:
- board text removed: "Made by: Manas Moondra Grant Gardner Yen Do Elliott Suh Brandon Mueller Daniel Phan"
