File: PCB/Compute_Module/CM4_Small breakout/Compute module small/CM4-NAS-MiniPCIE/CM4_2.kicad_pcb (KiCad board)
At the start: 4 copper layers, 90 x 75 mm, 23 parts, among them J10 PCIE_USB_D-/D+, J11 V_IN1, J12 V_IN2, J17 GPIO_V, J2 USB_A, J20 Controll Connector, J3 USB_HUB, J30 Conn_01x07_Female, J4 USB_B_Micro, J40 N_LED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

Commit message: 3/4 almost done
Parts:
- removed F1, F2: Polyfuse, Resistor_SMD:R_0805_2012Metric
- removed J10: PCIE_USB_D-/D+, Connector_PinHeader_2.54mm:PinHeader_1x02_P2.54mm_Vertical
- removed J11: V_IN1, Connector_PinHeader_2.54mm:PinHeader_1x04_P2.54mm_Vertical
- removed J12: V_IN2, Connector_PinHeader_2.54mm:PinHeader_1x04_P2.54mm_Vertical
- removed J20: Controll Connector, Connector_PinHeader_2.54mm:PinHeader_1x07_P2.54mm_Vertical
- removed J30: Conn_01x07_Female, Connector_PinSocket_2.54mm:PinSocket_1x07_P2.54mm_Vertical
- removed J42: 1V5, Connector_PinHeader_2.54mm:PinHeader_1x01_P2.54mm_Vertical
- removed J7: USB_OTG, Connector_PinHeader_2.54mm:PinHeader_1x02_P2.54mm_Vertical
- added K4: RASPBERRY_PI4_HEADER, e-radionica.com footprinti:RASPBERRY_PI4_HEADER, F.Cu at (568.6, 329.9)
- moved R6 30.0 mm to (540.7, 323.5), turned to 0 degrees
- moved R5 27.6 mm to (540.7, 325.6), turned to 0 degrees
- moved J8 22.6 mm to (547.5, 329.1)
Connections:
- Module1 pad 77: +5V_USB_IN -> 5V_CM4
- Module1 pad 79: +5V_USB_IN -> 5V_CM4
- Module1 pad 81: +5V_USB_IN -> 5V_CM4
- Module1 pad 83: +5V_USB_IN -> 5V_CM4
- Module1 pad 85: +5V_USB_IN -> 5V_CM4
- Module1 pad 87: +5V_USB_IN -> 5V_CM4
Routing:
- net +5V_USB: track 91.7 -> 4.57 mm, vias 8 -> 0
- net +5V_USB_IN: track 161.9 -> 119.0 mm
- net 1V5_PCIE: track 40.3 -> 0.00 mm, vias 2 -> 0
- net (no net): track 30.2 -> 0.00 mm, vias 8 -> 0
- net 3V3_PCIE: track 29.8 -> 0.00 mm
- net GPIO2: track 35.4 -> 5.96 mm
- net GPIO3: track 30.8 -> 4.57 mm
- net GPIO4: track 25.4 -> 0.90 mm, vias 1 -> 0
- net /PCIe_USB_D_N: track 22.3 -> 0.00 mm
- net /ID_SD: track 10.0 -> 25.4 mm
- net GPIO12: track 14.2 -> 3.67 mm
- net GPIO15: track 14.9 -> 4.94 mm
- net GPIO14: track 13.8 -> 4.18 mm
- net /PCIe_USB_D_P: track 7.46 -> 0.00 mm
- net /+3.3v: track 2.77 -> 8.16 mm
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Other:
- board text added: "3v3"
- board text added: "5V"
