File: PCB/Power_Regulator_12.6v_input/Power_Regulator_12.6v_input.kicad_pcb (KiCad board)
At the start: 2 copper layers, 90 x 90 mm, 54 parts, among them J1 SE2-30, U1 TLP3542, U2 TPS55340RTER, U3 TPS563203, U4 TPS54JA20RWWR

Commit message: edited trace widths and moved some stuff
Parts:
- moved C24 10.7 mm to (139.0, 69.5)
- moved C29 10.7 mm to (142.1, 69.5)
- moved C8 0.10 mm to (147.2, 108.5)
Routing:
- net Net-(U4-SW): track 12.8 -> 15.7 mm, vias 2 -> 6
- net +5V: track 65.3 -> 66.9 mm
- net Net-(U4-VCC): track 3.68 -> 2.15 mm

Commit message: edited trace widths and moved some stuff
Parts:
- removed R2: 20k, Resistor_SMD:R_0603_1608Metric
- R10: value 115k -> 135k
- moved R11 20.7 mm to (137.8, 89.1)
- moved R10 18.1 mm to (134.9, 89.9), turned to 90 degrees
- moved C14 6.95 mm to (140.6, 89.9)
- moved C10 6.42 mm to (147.0, 89.9)
- moved L3 6.13 mm to (122.8, 88.9)
- moved C33 5.48 mm to (132.8, 89.9)
- moved C13 3.13 mm to (140.4, 86.2), turned to 90 degrees
- moved C34 2.65 mm to (142.6, 89.9)
- moved C11 2.10 mm to (137.9, 81.0)
- moved C12 2.10 mm to (135.8, 81.0)
- moved C35 1.82 mm to (144.7, 89.9)
Connections:
- R10 pad 2: Net-(R10-Pad2) -> Net-(U3-FB)
Routing:
- net +3.3VA: track 97.9 -> 125.7 mm
- net Net-(U3-FB): track 33.1 -> 12.6 mm, vias 3 -> 2
- net Net-(U3-SW): track 10.7 -> 19.8 mm
- net Net-(U3-BST): track 4.60 -> 2.19 mm
- net Net-(R10-Pad2): track 2.05 -> 0.00 mm
- net Net-(U2-FB): track 20.3 -> 19.3 mm
- net GND: vias 113 -> 111
