File: PCB/Power_Regulator_12.6v_input/Power_Regulator_12.6v_input.kicad_pcb (KiCad board)
At the start: 2 copper layers, 90 x 83.5 mm, 65 parts, among them J1 SE2-30, J2 Jack-DC, J3 Conn_01x05_Pin, SW1 SW_SPDT_321, U1 TLP3542, U2 TPS55340RTER, U3 TPS563203, U4 TPS54JA20RWWR

Commit message: updated pcb to accomodate larger inductors, fixed swapped resistors
Parts:
- J10: renamed from 5v in to 3.3
- J12: renamed from Relay Logic
- J13: renamed from 3.3 relay logic input
- J5: renamed from 3.3V out
- J6: renamed from 24V pre Relay
- J8: renamed from +Batt 5v
- J9: renamed from +Batt 24v
- L2: value L8.2uH -> L10uH; footprint Inductor_SMD:L_0603_1608Metric -> SRR1208-100ML:IND_BOURNS_SRR1208
- L4: footprint Inductor_SMD:L_0603_1608Metric -> footprints:IND_IHLP-3232DZ_VIS-L
- R13: value R47.5k -> R60.4k
- renumbered +5V to J4, +24v to J7
