File: PCB/Power_Regulator_12.6v_input/Power_Regulator_12.6v_input.kicad_sch (KiCad schematic)
At the start: 55 parts, among them J1 SE2-30, J2 Jack-DC, U1 TLP3542, U2 TPS55340RTER, U3 TPS563203, U4 TPS54JA20RWWR

Commit message: connected all components and ran DRC with no errors
Parts:
- R1, R10, R11, R13, R14, R15, R16, R18, R19, R2, R20, R21, R22, R3, R4, R9: footprint Resistor_THT:R_Axial_DIN0207_L6.3mm_D2.5mm_P7.62mm_Horizontal -> Resistor_SMD:R_0603_1608Metric
Changed lines of the file:
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@@
 			)
 		)
-		(property "Footprint" "Resistor_THT:R_Axial_DIN0207_L6.3mm_D2.5mm_P7.62mm_Horizontal"
+		(property "Footprint" "Resistor_SMD:R_0603_1608Metric"
 			(at 193.802 121.92 90)
 			(effects
@@
 			)
 		)
-		(property "Footprint" "Resistor_THT:R_Axial_DIN0207_L6.3mm_D2.5mm_P7.62mm_Horizontal"
+		(property "Footprint" "Resistor_SMD:R_0603_1608Metric"
 			(at 39.37 184.15 0)
 			(effects
@@
 			)
 		)
-		(property "Footprint" "Resistor_THT:R_Axial_DIN0207_L6.3mm_D2.5mm_P7.62mm_Horizontal"
+		(property "Footprint" "Resistor_SMD:R_0603_1608Metric"
 			(at 64.008 128.27 90)
 			(effects
@@
 			)
 		)
-		(property "Footprint" "Resistor_THT:R_Axial_DIN0207_L6.3mm_D2.5mm_P7.62mm_Horizontal"
+		(property "Footprint" "Resistor_SMD:R_0603_1608Metric"
 			(at 242.062 115.57 90)
 			(effects
@@
 			)
 		)
-		(property "Footprint" "Resistor_THT:R_Axial_DIN0207_L6.3mm_D2.5mm_P7.62mm_Horizontal"
+		(property "Footprint" "Resistor_SMD:R_0603_1608Metric"
 			(at 80.772 78.74 90)
 			(effects
@@
 			)
 		)
-		(property "Footprint" "Resistor_THT:R_Axial_DIN0207_L6.3mm_D2.5mm_P7.62mm_Horizontal"
+		(property "Footprint" "Resistor_SMD:R_0603_1608Metric"
 			(at 242.062 124.46 90)
 			(effects
@@
 			)
 		)
-		(property "Footprint" "Resistor_THT:R_Axial_DIN0207_L6.3mm_D2.5mm_P7.62mm_Horizontal"
+		(property "Footprint" "Resistor_SMD:R_0603_1608Metric"
 			(at 149.352 41.91 90)
 			(effects
@@
 			)
 		)
-		(property "Footprint" "Resistor_THT:R_Axial_DIN0207_L6.3mm_D2.5mm_P7.62mm_Horizontal"
+		(property "Footprint" "Resistor_SMD:R_0603_1608Metric"
 			(at 149.352 52.07 90)
 			(effects
@@
 			)
 		)
-		(property "Footprint" "Resistor_THT:R_Axial_DIN0207_L6.3mm_D2.5mm_P7.62mm_Horizontal"
+		(property "Footprint" "Resistor_SMD:R_0603_1608Metric"
 			(at 27.94 180.34 0)
 			(effects
@@
 			)
 		)
-		(property "Footprint" "Resistor_THT:R_Axial_DIN0207_L6.3mm_D2.5mm_P7.62mm_Horizontal"
+		(property "Footprint" "Resistor_SMD:R_0603_1608Metric"
 			(at 68.072 76.2 90)
 			(effects
@@
 			)
 		)
-		(property "Footprint" "Resistor_THT:R_Axial_DIN0207_L6.3mm_D2.5mm_P7.62mm_Horizontal"
+		(property "Footprint" "Resistor_SMD:R_0603_1608Metric"
 			(at 117.602 125.73 90)
 			(effects
@@
 			)
 		)
-		(property "Footprint" "Resistor_THT:R_Axial_DIN0207_L6.3mm_D2.5mm_P7.62mm_Horizontal"
+		(property "Footprint" "Resistor_SMD:R_0603_1608Metric"
 			(at 240.03 130.302 90)
 			(effects
@@
 			)
 		)
-		(property "Footprint" "Resistor_THT:R_Axial_DIN0207_L6.3mm_D2.5mm_P7.62mm_Horizontal"
+		(property "Footprint" "Resistor_SMD:R_0603_1608Metric"
 			(at 58.42 138.938 90)
 			(effects
@@
 			)
 		)
-		(property "Footprint" "Resistor_THT:R_Axial_DIN0207_L6.3mm_D2.5mm_P7.62mm_Horizontal"
+		(property "Footprint" "Resistor_SMD:R_0603_1608Metric"
 			(at 117.602 138.43 90)
 			(effects
@@
 			)
 		)
-		(property "Footprint" "Resistor_THT:R_Axial_DIN0207_L6.3mm_D2.5mm_P7.62mm_Horizontal"
+		(property "Footprint" "Resistor_SMD:R_0603_1608Metric"
 			(at 78.232 60.96 90)
 			(effects
@@
 			)
 		)
-		(property "Footprint" "Resistor_THT:R_Axial_DIN0207_L6.3mm_D2.5mm_P7.62mm_Horizontal"
+		(property "Footprint" "Resistor_SMD:R_0603_1608Metric"
 			(at 68.072 49.53 90)
 			(effects

Commit message: edited trace widths and moved some stuff
Parts:
- removed R2: 20k, Resistor_SMD:R_0603_1608Metric, symbol Device:R
- R10: value 115k -> 135k
Connections:
- net at C33.2, R11.1, U3.6 (FB): now also R10.2
Other:
- moved on the sheet: R11
Changed lines of the file:
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@@
 	)
 	(junction
-		(at 243.84 129.54)
+		(at 243.84 123.19)
 		(diameter 0)
 		(color 0 0 0 0)
@@
 	(wire
 		(pts
-			(xy 243.84 119.38) (xy 243.84 120.65)
-		)
-		(stroke
-			(width 0)
-			(type default)
-		)
-	)
-	(wire
-		(pts
 			(xy 59.69 127) (xy 58.42 127)
 		)
@@
 	(wire
 		(pts
-			(xy 243.84 129.54) (xy 243.84 132.08)
+			(xy 243.84 123.19) (xy 243.84 125.73)
 		)
 		(stroke
@@
 	(wire
 		(pts
-			(xy 234.95 132.08) (xy 236.22 132.08)
+			(xy 234.95 125.73) (xy 236.22 125.73)
 		)
 		(stroke
@@
 	(wire
 		(pts
-			(xy 243.84 129.54) (xy 243.84 128.27)
+			(xy 243.84 119.38) (xy 243.84 123.19)
 		)
 		(stroke
@@
 	(wire
 		(pts
-			(xy 237.49 129.54) (xy 243.84 129.54)
+			(xy 237.49 123.19) (xy 243.84 123.19)
 		)
 		(stroke
@@
 	(wire
 		(pts
-			(xy 237.49 120.65) (xy 237.49 129.54)
+			(xy 237.49 120.65) (xy 237.49 123.19)
 		)
 		(stroke
@@
 			)
 		)
-		(property "Value" "115k"
+		(property "Value" "135k"
 			(at 246.38 116.8399 0)
 			(effects
@@
 	(symbol
 		(lib_id "power:GND")
-		(at 234.95 132.08 270)
+		(at 234.95 125.73 270)
 		(mirror x)
 		(unit 1)
@@
 		(fields_autoplaced yes)
 		(property "Reference" "#PWR0102"
-			(at 228.6 132.08 0)
+			(at 228.6 125.73 0)
 			(effects
 				(font
@@
 		)
 		(property "Value" "GND"
-			(at 231.14 132.0799 90)
+			(at 231.14 125.7299 90)
 			(effects
 				(font
@@
 		)
 		(property "Footprint" ""
-			(at 234.95 132.08 0)
+			(at 234.95 125.73 0)
 			(effects
 				(font
@@
 		)
 		(property "Datasheet" ""
-			(at 234.95 132.08 0)
+			(at 234.95 125.73 0)
 			(effects
 				(font
@@
 		)
 		(property "Description" "Power symbol creates a global label with name \"GND\" , ground"
-			(at 234.95 132.08 0)
+			(at 234.95 125.73 0)
 			(effects
 				(font
@@
 	)
 	(symbol
-		(lib_id "Device:R")
-		(at 243.84 124.46 0)
-		(unit 1)
-		(exclude_from_sim no)
-		(in_bom yes)
-		(on_board yes)
-		(dnp no)
-		(property "Reference" "R2"
-			(at 246.38 123.1899 0)
-			(effects
-				(font
-					(size 1.27 1.27)
-				)
-				(justify left)
-			)
-		)
-		(property "Value" "20k"
-			(at 246.38 125.7299 0)
-			(effects
-				(font
-					(size 1.27 1.27)
-				)
-				(justify left)
-			)
-		)
-		(property "Footprint" "Resistor_SMD:R_0603_1608Metric"
-			(at 242.062 124.46 90)
-			(effects
-				(font
-					(size 1.27 1.27)
-				)
-				(hide yes)
-			)
-		)
-		(property "Datasheet" "~"
-			(at 243.84 124.46 0)
-			(effects
-				(font
-					(size 1.27 1.27)
-				)
-				(hide yes)
-			)
-		)
-		(property "Description" "Resistor"
-			(at 243.84 124.46 0)
-			(effects
-				(font
-					(size 1.27 1.27)
-				)
-				(hide yes)
-			)
-		)
-		(pin "1"
-		)
-		(pin "2"
-		)
-		(instances
-			(project "Power_Regulator_12.6v_input"
-				(path "/3e19382a-168a-41e3-8127-b0b5a7558ca8"
-					(reference "R2")
-					(unit 1)
-				)
-			)
-		)
-	)
-	(symbol
 		(lib_id "power:+BATT")
 		(at 273.05 45.72 0)
@@
 	(symbol
 		(lib_id "Device:R")
-		(at 240.03 132.08 270)
+		(at 240.03 125.73 270)
 		(unit 1)
 		(exclude_from_sim no)
@@
 		(dnp no)
 		(property "Reference" "R11"
-			(at 241.3 133.858 0)
+			(at 241.3 127.508 0)
 			(effects
 				(font
@@
 		)
 		(property "Value" "30k"
-			(at 238.76 133.858 0)
+			(at 238.76 127.508 0)
 			(effects
 				(font
@@
 		)
 		(property "Footprint" "Resistor_SMD:R_0603_1608Metric"
-			(at 240.03 130.302 90)
+			(at 240.03 123.952 90)
 			(effects
 				(font
@@
 		)
 		(property "Datasheet" "~"
-			(at 240.03 132.08 0)
+			(at 240.03 125.73 0)
 			(effects
 				(font
@@
 		)
 		(property "Description" "Resistor"
-			(at 240.03 132.08 0)
+			(at 240.03 125.73 0)
 			(effects
 				(font
