File: PCB/Backplane/Backplane.kicad_pcb (KiCad board)
At the start: 2 copper layers, 10 parts, among them J1 5530843-7, J10 5530843-7, J2 5530843-7, J3 5530843-7, J4 5530843-7, J5 5530843-7, J6 5530843-7, J7 5530843-7, J8 5530843-7, J9 5530843-7

Commit message: edge cuts! thanks G2
Parts:
- removed J10, J9: 5530843-7, 5530843-7:TE_5530843-7
- moved J6 23.4 mm to (122.7, 147.0)
- moved J7 23.4 mm to (122.7, 181.0)
- moved J8 23.4 mm to (122.7, 215.0)
- moved J3 23.4 mm to (122.7, 45.0)
- moved J1 23.4 mm to (122.7, -23.0)
- moved J2 23.4 mm to (122.7, 11.0)
- moved J4 23.4 mm to (122.7, 79.0)
- moved J5 23.4 mm to (122.7, 113.0)
Routing:
- net /53: track 314.4 -> 244.5 mm
- net /31: track 314.4 -> 244.5 mm
- net /3: track 314.4 -> 244.5 mm
- net /7: track 314.4 -> 244.5 mm
- net /51: track 314.4 -> 244.5 mm
- net /24: track 314.4 -> 244.5 mm
- net /20: track 314.4 -> 244.5 mm
- net /12: track 314.4 -> 244.5 mm
- net /59: track 314.4 -> 244.5 mm
- net /39: track 314.4 -> 244.5 mm
- net /30: track 314.4 -> 244.5 mm
- net /17: track 314.4 -> 244.5 mm
- net /14: track 314.4 -> 244.5 mm
- net /49: track 314.4 -> 244.5 mm
- net /40: track 314.4 -> 244.5 mm
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Other:
- board outline added: 85 x 250 mm

Commit message: Updated backplane and removed unused connectors
Parts:
- added G***: LOGO, SC2-30:Rocketry_Logo_Symbol, B.Cu at (186.6, 146.5)
- moved J1 81.7 mm to (186.9, 27.5)
- moved J2 81.7 mm to (186.9, 61.5)
- moved J3 81.7 mm to (186.9, 95.5)
- moved J4 81.7 mm to (186.9, 129.5)
- moved J5 81.7 mm to (186.9, 163.5)
- moved J6 81.7 mm to (186.9, 197.5)
- moved J7 81.7 mm to (186.9, 231.5)
- moved J8 81.7 mm to (186.9, 265.5)
Other:
- board text added: "BACK"
- board text added: "FRONT"

Commit message: Finished new backplane
Parts:
- J1, J2, J3, J4, J5, J6, J7, J8: value 5530843-7 -> CONNECTOR-BACKPLANE
- moved J8 1.90 mm to (185.7, 267.0)
- moved J1 1.90 mm to (185.7, 29.0)
- moved J2 1.90 mm to (185.7, 63.0)
- moved J3 1.90 mm to (185.7, 97.0)
- moved J4 1.90 mm to (185.7, 131.0)
- moved J5 1.90 mm to (185.7, 165.0)
- moved J6 1.90 mm to (185.7, 199.0)
- moved J7 1.90 mm to (185.7, 233.0)
- moved G*** 1.70 mm to (185.7, 148.0)
Connections:
- J1 pad 23: /23 -> +3V3
- J1 pad 24: /24 -> +5V
- J1 pad 25: /25 -> +5V
- J1 pad 26: /26 -> +5V
- J1 pad 27: /27 -> VBUS
- J1 pad 28: /28 -> VBUS
- J1 pad 29: /29 -> GND
- J1 pad 30: /30 -> GND
- J1 pad 53: /53 -> +3V3
- J1 pad 54: /54 -> +5V
- J1 pad 55: /55 -> +5V
- J1 pad 56: /56 -> +5V
- J1 pad 57: /57 -> VBUS
- J1 pad 58: /58 -> VBUS
- J1 pad 59: /59 -> GND
- J1 pad 60: /60 -> GND
- J2 pad 23: /23 -> +3V3
- J2 pad 24: /24 -> +5V
- J2 pad 25: /25 -> +5V
- J2 pad 26: /26 -> +5V
- J2 pad 27: /27 -> VBUS
- J2 pad 28: /28 -> VBUS
- J2 pad 29: /29 -> GND
- J2 pad 30: /30 -> GND
- J2 pad 53: /53 -> +3V3
- J2 pad 54: /54 -> +5V
- J2 pad 55: /55 -> +5V
- J2 pad 56: /56 -> +5V
- J2 pad 57: /57 -> VBUS
- J2 pad 58: /58 -> VBUS
- J2 pad 59: /59 -> GND
- J2 pad 60: /60 -> GND
- J3 pad 23: /23 -> +3V3
- J3 pad 24: /24 -> +5V
- J3 pad 25: /25 -> +5V
- J3 pad 26: /26 -> +5V
- J3 pad 27: /27 -> VBUS
- J3 pad 28: /28 -> VBUS
- J3 pad 29: /29 -> GND
- J3 pad 30: /30 -> GND
- J3 pad 53: /53 -> +3V3
- J3 pad 54: /54 -> +5V
- J3 pad 55: /55 -> +5V
- J3 pad 56: /56 -> +5V
- J3 pad 57: /57 -> VBUS
- J3 pad 58: /58 -> VBUS
- J3 pad 59: /59 -> GND
- J3 pad 60: /60 -> GND
- J4 pad 23: /23 -> +3V3
- J4 pad 24: /24 -> +5V
- J4 pad 25: /25 -> +5V
- J4 pad 26: /26 -> +5V
- J4 pad 27: /27 -> VBUS
- J4 pad 28: /28 -> VBUS
- J4 pad 29: /29 -> GND
- J4 pad 30: /30 -> GND
- J4 pad 53: /53 -> +3V3
- J4 pad 54: /54 -> +5V
- J4 pad 55: /55 -> +5V
- J4 pad 56: /56 -> +5V
- J4 pad 57: /57 -> VBUS
- J4 pad 58: /58 -> VBUS
- J4 pad 59: /59 -> GND
- J4 pad 60: /60 -> GND
- J5 pad 23: /23 -> +3V3
- J5 pad 24: /24 -> +5V
- J5 pad 25: /25 -> +5V
- J5 pad 26: /26 -> +5V
- J5 pad 27: /27 -> VBUS
- J5 pad 28: /28 -> VBUS
- J5 pad 29: /29 -> GND
- J5 pad 30: /30 -> GND
- J5 pad 53: /53 -> +3V3
- J5 pad 54: /54 -> +5V
- J5 pad 55: /55 -> +5V
- J5 pad 56: /56 -> +5V
- J5 pad 57: /57 -> VBUS
- J5 pad 58: /58 -> VBUS
- J5 pad 59: /59 -> GND
- J5 pad 60: /60 -> GND
- J6 pad 23: /23 -> +3V3
- J6 pad 24: /24 -> +5V
- J6 pad 25: /25 -> +5V
- J6 pad 26: /26 -> +5V
- J6 pad 27: /27 -> VBUS
- J6 pad 28: /28 -> VBUS
- J6 pad 29: /29 -> GND
- J6 pad 30: /30 -> GND
- J6 pad 53: /53 -> +3V3
- J6 pad 54: /54 -> +5V
- J6 pad 55: /55 -> +5V
- J6 pad 56: /56 -> +5V
- J6 pad 57: /57 -> VBUS
- J6 pad 58: /58 -> VBUS
- J6 pad 59: /59 -> GND
- J6 pad 60: /60 -> GND
- J7 pad 23: /23 -> +3V3
- J7 pad 24: /24 -> +5V
- J7 pad 25: /25 -> +5V
- J7 pad 26: /26 -> +5V
- J7 pad 27: /27 -> VBUS
- J7 pad 28: /28 -> VBUS
- J7 pad 29: /29 -> GND
- J7 pad 30: /30 -> GND
- J7 pad 53: /53 -> +3V3
- J7 pad 54: /54 -> +5V
- J7 pad 55: /55 -> +5V
- J7 pad 56: /56 -> +5V
- J7 pad 57: /57 -> VBUS
- J7 pad 58: /58 -> VBUS
- J7 pad 59: /59 -> GND
- J7 pad 60: /60 -> GND
- J8 pad 23: /23 -> +3V3
- J8 pad 24: /24 -> +5V
- J8 pad 25: /25 -> +5V
- J8 pad 26: /26 -> +5V
- J8 pad 27: /27 -> VBUS
- J8 pad 28: /28 -> VBUS
- J8 pad 29: /29 -> GND
- J8 pad 30: /30 -> GND
- J8 pad 53: /53 -> +3V3
- J8 pad 54: /54 -> +5V
- J8 pad 55: /55 -> +5V
- J8 pad 56: /56 -> +5V
- J8 pad 57: /57 -> VBUS
- J8 pad 58: /58 -> VBUS
- J8 pad 59: /59 -> GND
- J8 pad 60: /60 -> GND
Routing:
- net /59: track 244.5 -> 0.00 mm
- net /60: track 244.5 -> 0.00 mm
- net /58: track 244.5 -> 0.00 mm
- net /24: track 244.5 -> 0.00 mm
- net /23: track 244.5 -> 0.00 mm
- net /30: track 244.5 -> 0.00 mm
- net /29: track 244.5 -> 0.00 mm
- net /57: track 244.5 -> 0.00 mm
- net /54: track 244.5 -> 0.00 mm
- net /56: track 244.5 -> 0.00 mm
- net /55: track 244.5 -> 0.00 mm
- net /28: track 244.5 -> 0.00 mm
- net /26: track 244.5 -> 0.00 mm
- net /53: track 244.5 -> 0.00 mm
- net /25: track 244.5 -> 0.00 mm
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- added copper zone on B.Cu, net +3V3
- added copper zone on F.Cu, net +3V3
- added copper zone on B.Cu, net +5V
- added copper zone on F.Cu, net +5V
- added copper zone on B.Cu, net GND
- added copper zone on F.Cu, net GND
- added copper zone on B.Cu, net VBUS
- added copper zone on F.Cu, net VBUS
Other:
- board text removed: "BACK"
- board text removed: "FRONT"

Commit message: Improved power rail layout and added silkscreen, added teardrops
Other:
- board text added: "+3V3"
- board text added: "+5V0"
- board text added: "Connector 1"
- board text added: "Connector 2"
- board text added: "Connector 3"
- board text added: "Connector 4"
- board text added: "Connector 5"
- board text added: "Connector 6"
- board text added: "Connector 7"
- board text added: "Connector 8"
- board text added: "GND"
- board text added: "Power Rails"
- board text added: "VBus"
- board text added: "↑ TOP ↑ BACK"
- board text added: "↑ TOP ↑ FRONT"

Commit message: Touched up spacing to make it exact
Routing:
- net /47: track 246.0 -> 245.4 mm
- net /36: track 246.0 -> 245.4 mm
- net /34: track 246.0 -> 245.4 mm
- net /32: track 246.0 -> 245.4 mm
- net /31: track 246.0 -> 245.4 mm
- net /52: track 246.0 -> 245.4 mm
- net /51: track 246.0 -> 245.4 mm
- net /50: track 246.0 -> 245.4 mm
- net /49: track 246.0 -> 245.4 mm
- net /46: track 246.0 -> 245.4 mm
- net /43: track 246.0 -> 245.4 mm
- net /42: track 246.0 -> 245.4 mm
- net /41: track 246.0 -> 245.4 mm
- net /38: track 246.0 -> 245.4 mm
- net /37: track 246.0 -> 245.4 mm
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