File: PCB/Backplane/Backplane.kicad_pcb (KiCad board)
At the start: 2 copper layers, 85 x 250 mm, 9 parts, among them J1 CONNECTOR-BACKPLANE, J2 CONNECTOR-BACKPLANE, J3 CONNECTOR-BACKPLANE, J4 CONNECTOR-BACKPLANE, J5 CONNECTOR-BACKPLANE, J6 CONNECTOR-BACKPLANE, J7 CONNECTOR-BACKPLANE, J8 CONNECTOR-BACKPLANE

Commit message: Added better labeling to backplane connectors
Other:
- board text added: "BOTTOM"
- board text added: "TOP"
- board text added: "↑ BACKPLANE TOP ↑ BACK"
- board text added: "↑ BACKPLANE TOP ↑ FRONT"
- board text removed: "↑ TOP ↑ BACK"
- board text removed: "↑ TOP ↑ FRONT"
Changed lines of the file:
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@@
+		)
+	)
+	(gr_text "TOP"
+		(at 227.1 90.1 0)
+		(layer "F.SilkS")
+		(effects
+			(font
+				(size 1.5 1.5)
+				(thickness 0.3)
+				(bold yes)
+			)
+			(justify right top)
+		)
+	)
+	(gr_text "TOP"
+		(at 227.1 226.1 0)
+		(layer "F.SilkS")
+		(effects
+			(font
+				(size 1.5 1.5)
+				(thickness 0.3)
+				(bold yes)
+			)
+			(justify right top)
+		)
+	)
+	(gr_text "BOTTOM"
+		(at 227.1 34.6 0)
+		(layer "F.SilkS")
+		(effects
+			(font
+				(size 1.5 1.5)
+				(thickness 0.3)
+				(bold yes)
+			)
+			(justify right top)
+		)
+	)
+	(gr_text "BOTTOM"
+		(at 227.1 204.6 0)
+		(layer "F.SilkS")
+		(effects
+			(font
+				(size 1.5 1.5)
+				(thickness 0.3)
+				(bold yes)
+			)
+			(justify right top)
+		)
+	)
+	(gr_text "TOP"
+		(at 227.1 192.1 0)
+		(layer "F.SilkS")
+		(effects
+			(font
+				(size 1.5 1.5)
+				(thickness 0.3)
+				(bold yes)
+			)
+			(justify right top)
 		)
 	)
@@
 		)
 	)
+	(gr_text "BOTTOM"
+		(at 227.1 136.6 0)
+		(layer "F.SilkS")
+		(effects
+			(font
+				(size 1.5 1.5)
+				(thickness 0.3)
+				(bold yes)
+			)
+			(justify right top)
+		)
+	)
 	(gr_text "Connector 5"
 		(at 144.5 170.5 0)
@@
 			)
 			(justify left top)
+		)
+	)
+	(gr_text "BOTTOM"
+		(at 227.1 68.6 0)
+		(layer "F.SilkS")
+		(effects
+			(font
+				(size 1.5 1.5)
+				(thickness 0.3)
+				(bold yes)
+			)
+			(justify right top)
 		)
 	)
@@
 		)
 	)
+	(gr_text "TOP"
+		(at 227.1 260.1 0)
+		(layer "F.SilkS")
+		(effects
+			(font
+				(size 1.5 1.5)
+				(thickness 0.3)
+				(bold yes)
+			)
+			(justify right top)
+		)
+	)
+	(gr_text "BOTTOM"
+		(at 227.1 102.6 0)
+		(layer "F.SilkS")
+		(effects
+			(font
+				(size 1.5 1.5)
+				(thickness 0.3)
+				(bold yes)
+			)
+			(justify right top)
+		)
+	)
 	(gr_text "+5V0"
 		(at 209.9 54.1 90)
@@
 		)
 	)
+	(gr_text "TOP"
+		(at 227.1 56.1 0)
+		(layer "F.SilkS")
+		(effects
+			(font
+				(size 1.5 1.5)
+				(thickness 0.3)
+				(bold yes)
+			)
+			(justify right top)
+		)
+	)
 	(gr_text "Connector 7"
 		(at 144.5 238.5 0)
@@
 			)
 			(justify left top)
+		)
+	)
+	(gr_text "BOTTOM"
+		(at 227.1 170.6 0)
+		(layer "F.SilkS")
+		(effects
+			(font
+				(size 1.5 1.5)
+				(thickness 0.3)
+				(bold yes)
+			)
+			(justify right top)
 		)
 	)
@@
 		)
 	)
-	(gr_text "↑ TOP ↑\n\nFRONT"
+	(gr_text "↑ BACKPLANE TOP ↑\n\nFRONT"
 		(at 185.7 38.9 0)
 		(layer "F.SilkS")
@@
 				(bold yes)
 			)
+		)
+	)
+	(gr_text "BOTTOM"
+		(at 227.1 238.6 0)
+		(layer "F.SilkS")
+		(effects
+			(font
+				(size 1.5 1.5)
+				(thickness 0.3)
+				(bold yes)
+			)
+			(justify right top)
 		)
 	)
@@
 			)
 			(justify left top)
+		)
+	)
+	(gr_text "TOP"
+		(at 227.1 158.1 0)
+		(layer "F.SilkS")
+		(effects
+			(font
+				(size 1.5 1.5)
+				(thickness 0.3)
+				(bold yes)
+			)
+			(justify right top)
+		)
+	)
+	(gr_text "TOP"
+		(at 227.1 124.1 0)
+		(layer "F.SilkS")
+		(effects
+			(font
+				(size 1.5 1.5)
+				(thickness 0.3)
+				(bold yes)
+			)
+			(justify right top)
 		)
 	)
@@
 		)
 	)
-	(gr_text "↑ TOP ↑\n\nBACK"
+	(gr_text "↑ BACKPLANE TOP ↑\n\nBACK"
 		(at 185.709793 38.890988 0)
 		(layer "B.SilkS")

Commit message: Made board thinner by 1.5mm, removed reference identifier on back artwork
Other:
- board size 85 x 250 mm -> 83.5 x 250 mm
