File: PCB/Compute_Module V1.1/CM4_2.kicad_pcb (KiCad board)
At the start: 4 copper layers, 90 x 90 mm, 14 parts, among them J1 SE2-30, J2 USB_A, J3 USB_HUB, J4 USB_B_Micro, J5 Micro_SD_Card, J6 HDMI_A_1.4, J8 Conn_01x22_Female, J9 RJ45, K4 RASPBERRY_PI4_HEADER

Commit message: progress
Connections:
- J6 pad 18: +5V_HDMI -> /5V
Routing:
- net /5V: track 0.00 -> 190.8 mm, vias 0 -> 6
- net SCL: track 0.00 -> 103.4 mm, vias 0 -> 2
- net SDA: track 0.00 -> 98.5 mm, vias 0 -> 2
- net /27: track 0.00 -> 94.8 mm, vias 0 -> 1
- net /17: track 0.00 -> 88.6 mm, vias 0 -> 1
- net 3V3: track 0.00 -> 86.7 mm, vias 0 -> 1
- net +5V_HDMI: track 82.7 -> 0.00 mm
- net /22: track 0.00 -> 81.9 mm, vias 0 -> 2
- net /11: track 0.00 -> 75.5 mm, vias 0 -> 1
- net /14: track 0.00 -> 71.7 mm, vias 0 -> 1
- net /23: track 0.00 -> 68.2 mm, vias 0 -> 1
- net /15: track 0.00 -> 68.2 mm, vias 0 -> 1
- net /9: track 0.00 -> 66.1 mm, vias 0 -> 1
- net /18: track 0.00 -> 66.1 mm, vias 0 -> 1
- net /CAM_GPIO: track 0.00 -> 60.3 mm, vias 0 -> 2
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Other:
- board text removed: "Pinout on backside"

Commit message: Progress
Connections:
- J1 pad 33: unconnected-(J1-GPIO_4-Pad33) -> /4
- K4 pad 7: Net-(K4-GPIO4) -> /4
- Module1 pad 24: unconnected-(Module1A-GPIO26-Pad24) -> /26
- Module1 pad 25: unconnected-(Module1A-GPIO21-Pad25) -> /21
- Module1 pad 26: unconnected-(Module1A-GPIO19-Pad26) -> /19
- Module1 pad 27: unconnected-(Module1A-GPIO20-Pad27) -> /20
- Module1 pad 28: unconnected-(Module1A-GPIO13-Pad28) -> /13
- Module1 pad 29: unconnected-(Module1A-GPIO16-Pad29) -> /16
- Module1 pad 30: unconnected-(Module1A-GPIO6-Pad30) -> /6
- Module1 pad 31: GPIO12 -> /12
- Module1 pad 34: unconnected-(Module1A-GPIO5-Pad34) -> /5
- Module1 pad 37: unconnected-(Module1A-GPIO7-Pad37) -> /7
- Module1 pad 38: unconnected-(Module1A-GPIO11-Pad38) -> /11
- Module1 pad 39: unconnected-(Module1A-GPIO8-Pad39) -> /8
- Module1 pad 40: unconnected-(Module1A-GPIO9-Pad40) -> /9
- Module1 pad 41: unconnected-(Module1A-GPIO25-Pad41) -> /25
- Module1 pad 44: unconnected-(Module1A-GPIO10-Pad44) -> /10
- Module1 pad 45: unconnected-(Module1A-GPIO24-Pad45) -> /24
- Module1 pad 46: unconnected-(Module1A-GPIO22-Pad46) -> /22
- Module1 pad 47: unconnected-(Module1A-GPIO23-Pad47) -> /23
- Module1 pad 48: unconnected-(Module1A-GPIO27-Pad48) -> /27
- Module1 pad 49: unconnected-(Module1A-GPIO18-Pad49) -> /18
- Module1 pad 50: unconnected-(Module1A-GPIO17-Pad50) -> /17
- Module1 pad 51: GPIO15 -> /15
- Module1 pad 54: GPIO4 -> /4
- Module1 pad 55: GPIO14 -> /14
- Module1 pad 56: GPIO3 -> SCL
- Module1 pad 58: GPIO2 -> SDA
Routing:
- net /4: track 0.00 -> 150.8 mm, vias 0 -> 5
- net SCL: track 103.4 -> 224.0 mm, vias 2 -> 5
- net /6: track 45.1 -> 163.8 mm, vias 2 -> 8
- net /24: track 58.1 -> 172.9 mm, vias 1 -> 5
- net /5: track 48.6 -> 162.5 mm, vias 2 -> 6
- net /15: track 68.2 -> 174.1 mm, vias 1 -> 4
- net /7: track 56.4 -> 156.6 mm, vias 1 -> 2
- net /16: track 46.9 -> 144.6 mm, vias 1 -> 6
- net /12: track 51.1 -> 147.9 mm, vias 1 -> 3
- net /18: track 66.1 -> 162.7 mm, vias 1 -> 2
- net /14: track 71.7 -> 167.1 mm, vias 1 -> 3
- net /25: track 59.2 -> 152.6 mm, vias 1 -> 3
- net /20: track 45.3 -> 136.6 mm, vias 1 -> 4
- net SDA: track 98.5 -> 188.1 mm, vias 2 -> 5
- net /10: track 60.1 -> 147.5 mm, vias 1 -> 4
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