File: PCB/Compute_Module V1.1/CM4_2.kicad_sch (KiCad schematic)
At the start: 23 parts, among them J17 GPIO_V, J2 USB_A, J20 Controll Connector, J3 USB_HUB, J30 Conn_01x07_Female, J4 USB_B_Micro, J40 N_LED, J42 1V5, J5 Micro_SD_Card, J6 HDMI_A_1.4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

Commit message: 3/4 almost done
Parts:
- removed J17: GPIO_V, Connector_PinHeader_2.54mm:PinHeader_1x03_P2.54mm_Vertical_SMD_Pin1Right, symbol Connector_Generic:Conn_01x03
- removed J20: Controll Connector, Connector_PinHeader_2.54mm:PinHeader_1x07_P2.54mm_Vertical, symbol Connector:Conn_01x07_Female
- removed J30: Conn_01x07_Female, Connector_PinSocket_2.54mm:PinSocket_1x07_P2.54mm_Vertical, symbol Connector:Conn_01x07_Female
- removed J40: N_LED, Connector_PinHeader_2.54mm:PinHeader_1x01_P2.54mm_Vertical, symbol Connector_Generic:Conn_01x01
- removed J42: 1V5, Connector_PinHeader_2.54mm:PinHeader_1x01_P2.54mm_Vertical, symbol Connector_Generic:Conn_01x01
- removed J7: USB_OTG, Connector_PinHeader_2.54mm:PinHeader_1x02_P2.54mm_Vertical, symbol Connector:Conn_01x02_Male
- added J1: SE2-30, SE2-30:SE2-30, symbol SE2-30:SE2-30
- J9: footprint Connector_RJ:RJ45_Ninigi_GE -> Connector_RJ:RJ45_OST_PJ012-8P8CX_Vertical
Connections:
- net 3V3: now also J1.23 (3.3V), J1.53 (3.3V)
- net GND: now also J1.29 (GND), J1.30 (GND), J1.59 (GND), J1.60 (GND)
- net SCL: now also J1.32 (GPIO_3)
- net SDA: now also J1.31 (GPIO_2)
- net 15: now reaches K4.10 (GPIO15), K5.6
- net 15: now also J1.2 (GPIO_15)
- net 17: now reaches K1.5, K4.11 (GPIO17)
- net 17: now also J1.34 (GPIO_17)
- net 18: now reaches K4.12 (GPIO18), K5.5
- net 18: now also J1.3 (GPIO_18)
- net 27: now reaches K1.4, K4.13 (GPIO27)
- net 27: now also J1.35 (GPIO_27)
- net 22: now reaches K1.3, K4.15 (GPIO22)
- net 22: now also J1.36 (GPIO_22)
- net 23: now reaches K4.16 (GPIO23), K5.3
- net 23: now also J1.4 (GPIO_23)
- net 24: now reaches K4.18 (GPIO24), K5.2
- net 24: now also J1.5 (GPIO_24)
- net 10: now reaches K1.1, K4.19 (GPIO10)
- net 10: now also J1.37 (GPIO_10)
- net 5V: now reaches K4.2 (5V), K4.4 (5V), K5.10, K5.9
- net 5V: now also J1.24 (5V), J1.25 (5V), J1.26 (5V), J1.54 (5V), J1.55 (5V), J1.56 (5V)
- net 9: now reaches K2.10, K4.21 (GPIO9)
- net 9: now also J1.38 (GPIO_9)
- net 25: now reaches K4.22 (GPIO25), K6.10
- net 25: now also J1.6 (GPIO_25)
- net 11: now reaches K2.9, K4.23 (GPIO11)
- net 11: now also J1.39 (GPIO_11)
- net 8: now reaches K4.24 (GPIO8), K6.9
- net 8: now also J1.7 (GPIO_8)
- net 7: now reaches K4.26 (GPIO7), K6.8
- net 7: now also J1.8 (GPIO_7)
- net 0: now reaches K2.7, K4.27 (GPIO0)
- net 0: now also J1.40 (GPIO_0)
- net 1: now reaches K4.28 (GPIO1), K6.7
- net 1: now also J1.9 (GPIO_1)
- net 5: now reaches K2.6, K4.29 (GPIO5)
- net 5: now also J1.41 (GPIO_5)
- net 6: now reaches K2.5, K4.31 (GPIO6)
- net 6: now also J1.42 (GPIO_6)
- net 12: now reaches K4.32 (GPIO12), K6.5
- net 12: now also J1.10 (GPIO_12)
- net 13: now reaches K2.4, K4.33 (GPIO13)
- net 13: now also J1.43 (GPIO_13)
- net 19: now reaches K2.3, K4.35 (GPIO19)
- net 19: now also J1.44 (GPIO_19)
- net 16: now reaches K4.36 (GPIO16), K6.3
- net 16: now also J1.11 (GPIO_16)
- net 26: now reaches K2.2, K4.37 (GPIO26)
- net 26: now also J1.45 (GPIO_26)
- net 20: now reaches K4.38 (GPIO20), K6.2
- net 20: now also J1.12 (GPIO_20)
- net 21: now reaches K4.40 (GPIO21), K6.1
- net 21: now also J1.13 (GPIO_21)
- net 14: now reaches K4.8 (GPIO14), K5.7
- net 14: now also J1.1 (GPIO_14)
Other:
- note added: "Ethernet Vertical"
- note added: "SE2 Thingy Connector"
- note removed: "Connections"
- note removed: "Ethernet"
- moved on the sheet: K1, K2, K4, K5, K6, R5, R6

Commit message: Progress
Connections:
- net +5V_HDMI is gone; now on net 5V: J6.18 (+5V)
- net GPIO12 is gone; now on net 12: Module1.31 (GPIO12)
- net GPIO14 is gone; now on net 14: Module1.55 (GPIO14)
- net GPIO15 is gone; now on net 15: Module1.51 (GPIO15)
- net GPIO2 is gone; now on net SDA: Module1.58 (GPIO2)
- net GPIO3 is gone; now on net SCL: Module1.56 (GPIO3)
- net GPIO4 is gone; now on net 4: Module1.54 (GPIO4)
- net 10: now also Module1.44 (GPIO10)
- net 11: now also Module1.38 (GPIO11)
- net 13: now also Module1.28 (GPIO13)
- net 16: now also Module1.29 (GPIO16)
- net 17: now also Module1.50 (GPIO17)
- net 18: now also Module1.49 (GPIO18)
- net 19: now also Module1.26 (GPIO19)
- net 20: now also Module1.27 (GPIO20)
- net 21: now also Module1.25 (GPIO21)
- net 22: now also Module1.46 (GPIO22)
- net 23: now also Module1.47 (GPIO23)
- net 24: now also Module1.45 (GPIO24)
- net 25: now also Module1.41 (GPIO25)
- net 26: now also Module1.24 (GPIO26)
- net 27: now also Module1.48 (GPIO27)
- net 5: now also Module1.34 (GPIO5)
- net 6: now also Module1.30 (GPIO6)
- net 7: now also Module1.37 (GPIO7)
- net 8: now also Module1.39 (GPIO8)
- net 9: now also Module1.40 (GPIO9)
- net 4: now reaches K1.7, K4.7 (GPIO4)
- net 4: now also J1.33 (GPIO_4)
